Commit message: delete one file

File: urdf/lego/1_2x2.urdf (robot description, URDF)
Before this commit: robot Assem1, 1 links, 0 joints
Links:
- link base_link: mass 0.014644 -> 0.0024405; geometry collision mesh filename=urdf/lego_meshes/2x2.STL; visual mesh filename=urdf/lego_meshes/2x2.STL

File: urdf/lego/1_2x3.urdf (robot description, URDF)
Before this commit: robot 2x2, 1 links, 0 joints
Links:
- link base_link: mass 0.01 -> 0.0037381; geometry collision mesh filename=urdf/lego_meshes/2x3.STL; visual mesh filename=urdf/lego_meshes/2x3.STL

File: urdf/lego/1_2x4.urdf (robot description, URDF)
Before this commit: robot 2x3, 1 links, 0 joints
Links:
- link base_link: mass 0.01 -> 0.0053446; geometry collision mesh filename=urdf/lego_meshes/2x4.STL; visual mesh filename=urdf/lego_meshes/2x4.STL

File: urdf/lego/2_2x2.urdf (robot description, URDF)
Before this commit: robot Assem1, 1 links, 0 joints
Links:
- removed link base_link
- added link crayon, mass 0.014644; collision mesh filename=urdf/lego_meshes/crayon.STL; visual mesh filename=urdf/lego_meshes/crayon.STL

File: urdf/lego/2_2x3.urdf (robot description, URDF)
Before this commit: robot Assem1, 1 links, 0 joints
Links:
- removed link base_link
- added link crayon, mass 0.014644; collision mesh filename=urdf/lego_meshes/crayon.STL; visual mesh filename=urdf/lego_meshes/crayon.STL

File: urdf/lego/2_2x4.urdf (robot description, URDF)
Before this commit: robot 2x4, 1 links, 0 joints
Links:
- removed link base_link
- added link crayon, mass 0.014644; collision mesh filename=urdf/lego_meshes/crayon.STL; visual mesh filename=urdf/lego_meshes/crayon.STL

File: urdf/lego/2x2.urdf (robot description, URDF)
Before this commit: robot 2x2, 1 links, 0 joints
Links:
- link base_link: mass 0.01 -> 0.0024405; geometry collision mesh filename=urdf/lego_meshes/2x2.STL; visual mesh filename=urdf/lego_meshes/2x2.STL

File: urdf/lego/2x3.urdf (robot description, URDF)
Before this commit: robot 2x4, 1 links, 0 joints
Links:
- link base_link: mass 0.01 -> 0.0037381; geometry collision mesh filename=urdf/lego_meshes/2x3.STL; visual mesh filename=urdf/lego_meshes/2x3.STL

File: urdf/lego/2x4.urdf (robot description, URDF)
Before this commit: robot cra, 1 links, 0 joints
Links:
- removed link crayon
- added link base_link, mass 0.0053446; collision mesh filename=urdf/lego_meshes/2x4.STL; visual mesh filename=urdf/lego_meshes/2x4.STL
